File: CherryShield/cherryKeyShield.sch (EAGLE design)
At the start: 19 parts

Commit message: newer layout
Parts:
- removed B1: ARDUINO_UNO_R3_SHIELDBASIC, SparkFun-Boards:ARDUINO_UNO_R3_SHIELDBASIC
Connections:
- net X0: no longer B1.*D11
- net X1: no longer B1.D12
- net X2: no longer B1.D13
- net Y0: no longer B1.D8
- net Y1: no longer B1.*D9
- net Y2: no longer B1.*D10
Changed lines of the file:
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@@
 <?xml version="1.0" encoding="utf-8"?>
 <!DOCTYPE eagle SYSTEM "eagle.dtd">
-<eagle version="8.1.1">
+<eagle version="8.2.0">
 <drawing>
 <settings>
@@
 <part name="S5" library="SparkFun-Switches" deviceset="MOMENTARY-SWITCH-SPST-LED" device="-PTH-CHERRY"/>
 <part name="S6" library="SparkFun-Switches" deviceset="MOMENTARY-SWITCH-SPST-LED" device="-PTH-CHERRY"/>
-<part name="B1" library="SparkFun-Boards" deviceset="ARDUINO_UNO_R3_SHIELD" device="BASIC"/>
 <part name="D1" library="SparkFun-DiscreteSemi" deviceset="DIODE" device="-BAS16J" value="250mA/100V"/>
 <part name="D2" library="SparkFun-DiscreteSemi" deviceset="DIODE" device="-BAS16J" value="250mA/100V"/>
@@
 <part name="S8" library="SparkFun-Switches" deviceset="MOMENTARY-SWITCH-SPST-LED" device="-PTH-CHERRY"/>
 <part name="S9" library="SparkFun-Switches" deviceset="MOMENTARY-SWITCH-SPST-LED" device="-PTH-CHERRY"/>
-<part name="SUPPLY1" library="supply2" deviceset="GND" device=""/>
-<part name="P+1" library="supply1" deviceset="VCC" device=""/>
 </parts>
 <sheets>
@@
 <instance part="S5" gate="G$1" x="60.96" y="81.28" rot="R90"/>
 <instance part="S6" gate="G$1" x="91.44" y="81.28" rot="R90"/>
-<instance part="B1" gate="G$1" x="154.94" y="60.96"/>
 <instance part="D1" gate="G$1" x="27.94" y="104.14" rot="R270"/>
 <instance part="D2" gate="G$1" x="58.42" y="104.14" rot="R270"/>
@@
 <instance part="S8" gate="G$1" x="60.96" y="45.72" rot="R90"/>
 <instance part="S9" gate="G$1" x="88.9" y="45.72" rot="R90"/>
-<instance part="SUPPLY1" gate="GND" x="137.16" y="33.02"/>
-<instance part="P+1" gate="VCC" x="137.16" y="96.52"/>
 </instances>
 <busses>
@@
 <label x="43.18" y="116.84" size="1.778" layer="95"/>
 </segment>
-<segment>
-<pinref part="B1" gate="G$1" pin="*D11"/>
-<wire x1="167.64" y1="48.26" x2="175.26" y2="48.26" width="0.1524" layer="91"/>
-<label x="172.72" y="48.26" size="1.778" layer="95"/>
-</segment>
 </net>
 <net name="Y0" class="0">
@@
 <wire x1="88.9" y1="101.6" x2="88.9" y2="99.06" width="0.1524" layer="91"/>
 <junction x="88.9" y="99.06"/>
-</segment>
-<segment>
-<pinref part="B1" gate="G$1" pin="D8"/>
-<wire x1="167.64" y1="55.88" x2="175.26" y2="55.88" width="0.1524" layer="91"/>
-<label x="172.72" y="55.88" size="1.778" layer="95"/>
 </segment>
 </net>
@@
 <label x="45.72" y="66.04" size="1.778" layer="95"/>
 </segment>
-<segment>
-<pinref part="B1" gate="G$1" pin="*D9"/>
-<wire x1="167.64" y1="53.34" x2="175.26" y2="53.34" width="0.1524" layer="91"/>
-<label x="172.72" y="53.34" size="1.778" layer="95"/>
-</segment>
 </net>
 <net name="Y2" class="0">
@@
 <wire x1="86.36" y1="30.48" x2="86.36" y2="27.94" width="0.1524" layer="91"/>
 <junction x="86.36" y="27.94"/>
-</segment>
-<segment>
-<pinref part="B1" gate="G$1" pin="*D10"/>
-<wire x1="167.64" y1="50.8" x2="175.26" y2="50.8" width="0.1524" layer="91"/>
-<label x="172.72" y="50.8" size="1.778" layer="95"/>
 </segment>
 </net>
@@
 <label x="73.66" y="116.84" size="1.778" layer="95"/>
 </segment>
-<segment>
-<pinref part="B1" gate="G$1" pin="D12"/>
-<wire x1="167.64" y1="45.72" x2="175.26" y2="45.72" width="0.1524" layer="91"/>
-<label x="172.72" y="45.72" size="1.778" layer="95"/>
-</segment>
 </net>
 <net name="X2" class="0">
@@
 <label x="101.6" y="116.84" size="1.778" layer="95"/>
 </segment>
-<segment>
-<pinref part="B1" gate="G$1" pin="D13"/>
-<wire x1="167.64" y1="43.18" x2="175.26" y2="43.18" width="0.1524" layer="91"/>
-<label x="172.72" y="43.18" size="1.778" layer="95"/>
-</segment>
-</net>
+</net>
